Commit message: wip: add gripper center position

File: robotiq_2finger_grippers/robotiq_2f_140_gripper_visualization/urdf/robotiq_arg2f_140_model_macro.xacro (robot description, xacro)
@@ -213,3 +213,26 @@
     <xacro:robotiq_arg2f_gazebo prefix="${prefix}"/>
   </xacro:macro>
+  <xacro:macro name="robotiq_arg2f_140" params="prefix">
+    <xacro:robotiq_arg2f_base_link prefix="${prefix}"/>
+    <xacro:finger_links prefix="${prefix}" fingerprefix="left" stroke="140"/>
+    <xacro:finger_links prefix="${prefix}" fingerprefix="right" stroke="140"/>
+    <xacro:finger_joint prefix="${prefix}"/>
+    <xacro:right_outer_knuckle_joint prefix="${prefix}"/>
+    <xacro:robotiq_arg2f_transmission prefix="${prefix}"/>
+    <xacro:robotiq_arg2f_gazebo prefix="${prefix}"/>
+  </xacro:macro>
+  <link
+    name="link_grasp_center">
+  </link>
+  <joint
+    name="joint_grasp_center"
+    type="fixed">
+    <origin
+      xyz="0 0 0.2"
+      rpy="0 0 0" />
+    <parent
+      link="robotiq_arg2f_base_link" />
+    <child
+      link="link_grasp_center" />
+  </joint>
 </robot>
