Commit message: fix: stop arm from shaking

File: robotiq_2finger_grippers/robotiq_2f_140_gripper_visualization/urdf/robotiq_arg2f.gazebo.xacro (robot description, xacro)
@@ -34,4 +34,19 @@
             </plugin>
         </gazebo>
+        <gazebo reference="${prefix}right_outer_knuckle_joint">
+          <material value="Gazebo/White"/>
+        </gazebo>
+        <gazebo reference="${prefix}left_inner_knuckle_joint">
+          <material value="Gazebo/White"/>
+        </gazebo>
+        <gazebo reference="${prefix}right_inner_knuckle_joint">
+        <material value="Gazebo/White"/>
+        </gazebo>
+        <gazebo reference="${prefix}left_inner_finger_joint">
+        <material value="Gazebo/White"/>
+        </gazebo>
+        <gazebo reference="${prefix}right_inner_finger_joint">
+          <material value="Gazebo/White"/>
+        </gazebo>
     </xacro:macro>
 </robot>

Commit message: wip: change color to black and correct gazebo link

File: robotiq_2finger_grippers/robotiq_2f_140_gripper_visualization/urdf/robotiq_arg2f.gazebo.xacro (robot description, xacro)
@@ -34,18 +34,33 @@
             </plugin>
         </gazebo>
-        <gazebo reference="${prefix}right_outer_knuckle_joint">
-          <material value="Gazebo/White"/>
+        <gazebo reference="${prefix}right_outer_knuckle">
+          <material value="Gazebo/Black"/>
         </gazebo>
-        <gazebo reference="${prefix}left_inner_knuckle_joint">
-          <material value="Gazebo/White"/>
+        <gazebo reference="${prefix}left_outer_knuckle">
+          <material value="Gazebo/Black"/>
         </gazebo>
-        <gazebo reference="${prefix}right_inner_knuckle_joint">
-        <material value="Gazebo/White"/>
+        <gazebo reference="${prefix}right_inner_knuckle">
+        <material value="Gazebo/Black"/>
         </gazebo>
-        <gazebo reference="${prefix}left_inner_finger_joint">
-        <material value="Gazebo/White"/>
+        <gazebo reference="${prefix}left_inner_knuckle">
+          <material value="Gazebo/Black"/>
         </gazebo>
-        <gazebo reference="${prefix}right_inner_finger_joint">
-          <material value="Gazebo/White"/>
+        <gazebo reference="${prefix}left_inner_finger">
+        <material value="Gazebo/Black"/>
+        </gazebo>
+        <gazebo reference="${prefix}right_inner_finger">
+          <material value="Gazebo/Black"/>
+        </gazebo>
+        <gazebo reference="${prefix}left_outer_finger">
+          <material value="Gazebo/Black"/>
+        </gazebo>
+        <gazebo reference="${prefix}right_outer_finger">
+          <material value="Gazebo/Black"/>
+        </gazebo>
+        <gazebo reference="${prefix}right_inner_finger_pad">
+          <material value="Gazebo/Black"/>
+        </gazebo>
+        <gazebo reference="${prefix}left_inner_finger_pad">
+          <material value="Gazebo/Black"/>
         </gazebo>
     </xacro:macro>

File: robotiq_2finger_grippers/robotiq_2f_140_gripper_visualization/urdf/robotiq_arg2f.xacro (robot description, xacro)
@@ -24,4 +24,7 @@
       </collision>
     </link>
+    <gazebo reference="${prefix}robotiq_arg2f_base_link">
+      <material value="Gazebo/Black"/>
+    </gazebo>
   </xacro:macro>
   <xacro:macro name="finger_joints" params="prefix fingerprefix reflect">
