Commit message: wip: change gripper to black to ensure gazebo is reading correctly

File: robotiq_2finger_grippers/robotiq_2f_140_gripper_visualization/urdf/robotiq_arg2f.xacro (robot description, xacro)
@@ -5,6 +5,10 @@
       <inertial>
         <origin xyz="8.625E-08 -4.6583E-06 0.03145" rpy="0 0 0" />
-        <mass value="0.22652" />
-        <inertia ixx="0.00020005" ixy="-4.2442E-10" ixz="-2.9069E-10" iyy="0.00017832" iyz="-3.4402E-08" izz="0.00013478" />
+          <mass value="0.1" />
+          <inertia ixx="1.66667e-7" ixy="0.0" ixz="0.0"
+                   iyy="8.33333e-4" iyz="0.0"
+                   izz="8.33333e-4" />
+        <!-- <mass value="0.22652" /> -->
+        <!-- <inertia ixx="0.00020005" ixy="-4.2442E-10" ixz="-2.9069E-10" iyy="0.00017832" iyz="-3.4402E-08" izz="0.00013478" /> -->
       </inertial>
       <visual>

File: robotiq_2finger_grippers/robotiq_2f_140_gripper_visualization/urdf/robotiq_arg2f_140_model_macro.xacro (robot description, xacro)
@@ -126,4 +126,15 @@
   <xacro:macro name="inner_finger_pad" params="prefix fingerprefix">
     <link name="${prefix}${fingerprefix}_inner_finger_pad">
+      <inertial>
+        <origin xyz="0.000299999999999317 0.0160078233491243 -0.0136945669206257" rpy="0 0 0" />
+        <mass value="0.0104003125914103" />
+        <inertia
+            ixx="2.71909453810972E-06"
+            ixy="1.35402465472579E-21"
+            ixz="-7.1817349065269E-22"
+            iyy="7.69100314106116E-07"
+            iyz="6.74715432769696E-07"
+            izz="2.30315190420171E-06" />
+      </inertial>
       <visual>
         <origin xyz="0 0 0" rpy="0 0 0" />
